File: flip_dot_clock/flip_dot_clock.sch (KiCad schematic (older format))
At the start: 11 parts, among them J0 SWD Header, U0 TPS62177DQC, U1 STM32F070F6Px, U2 NCV7719

Commit message: add datasheets
Parts:
- C?: symbol mio:UCD1V101MNL1GS -> flip_dot_clock-rescue:UCD1V101MNL1GS-mio
- DS0: symbol mio:Small_7_Seg_FlipDot -> flip_dot_clock-rescue:Small_7_Seg_FlipDot-mio
- U2: symbol mio:NCV7719 -> flip_dot_clock-rescue:NCV7719-mio
Changed lines of the file:
@@
 EESchema Schematic File Version 4
-EELAYER 29 0
+EELAYER 30 0
 EELAYER END
 $Descr A4 11693 8268
@@
 $EndComp
 $Comp
-L mio:NCV7719 U2
+L flip_dot_clock-rescue:NCV7719-mio U2
 U 1 1 5CEE231A
 P 5800 2750
@@
 	5200 4750 5200 5050
 $Comp
-L mio:Small_7_Seg_FlipDot DS0
+L flip_dot_clock-rescue:Small_7_Seg_FlipDot-mio DS0
 U 1 1 5D1F5028
 P 5600 3950
@@
 	4850 3800 4850 2500
 $Comp
-L mio:UCD1V101MNL1GS C?
+L flip_dot_clock-rescue:UCD1V101MNL1GS-mio C?
 U 1 1 5D3C5739
 P 6350 1800

Commit message: update MCU. update kicad project.
Parts:
- removed U1: STM32F070F6Px, Package_SO:TSSOP-20_4.4x6.5mm_P0.65mm, symbol MCU_ST_STM32F0:STM32F070F6Px
- added U?: DS3231M, Package_SO:SOIC-16W_7.5x10.3mm_P1.27mm, symbol Timer_RTC:DS3231M
- added U?: STM32F051R8Tx, Package_QFP:LQFP-64_10x10mm_P0.5mm, symbol MCU_ST_STM32F0:STM32F051R8Tx
Connections:
- net labels added: +BATT, -BATT, I2C_SCL, I2C_SDA
- wire segments 125 -> 143
Other:
- moved on the sheet: C0, J0, L0, R0, U0
