File: kicad/control/flip_dot_clock.sch (KiCad schematic (older format))
At the start: 8 parts, among them U0 TPS62177DQC, U2 NCV7719

Commit message: add parts
Parts:
- removed C0: 22uF, symbol Device:C
- removed DS0: Small_7_Seg_FlipDot, symbol mio:Small_7_Seg_FlipDot
- removed L0: 10uH, symbol Device:L
- removed R0: 100k, symbol Device:R
- removed U0: TPS62177DQC, Package_SON:WSON-10-1EP_2x3mm_P0.5mm_EP0.84x2.4mm_ThermalVias, symbol Regulator_Switching:TPS62177DQC
- added J? (x2): Conn_01x15_Female, symbol Connector:Conn_01x15_Female
- U2: symbol mio:NCV7719 -> flip_dot_clock-rescue:NCV7719-mio
Connections:
- net labels removed: +24V
- wire segments 100 -> 39

Commit message: update schem
Parts:
- removed D?: MRA4003T3G, Diode_SMD:D_SMA, symbol Diode:MRA4003T3G
- removed J? (x2): Conn_01x15_Female, symbol Connector:Conn_01x15_Female
- removed U2: NCV7719, mio:SSOP-24_6.4x7.55mm_P0.65mm, symbol flip_dot_clock-rescue:NCV7719-mio
- removed U?: DS3231M, Package_SO:SOIC-16W_7.5x10.3mm_P1.27mm, symbol Timer_RTC:DS3231M
- added U?: NUCLEO-F303K8-HEADER, symbol mio:NUCLEO-F303K8-HEADER
- added U?: NCV7719, mio:SSOP-24_6.4x7.55mm_P0.65mm, symbol flip_dot_clock-rescue:NCV7719-mio
- added U?: Small_7_Seg_FlipDot_Module, symbol mio:Small_7_Seg_FlipDot_Module
- added U?: SLC03B-05, symbol mio:SLC03B-05
Connections:
- net labels added: +24V, +5V, A_SET_1, B_SET_1, C_SET_1, D_SET_1, E_SET_1, F_SET_1, G_SET_1, RESET_1, SPI1_CS_0, SPI1_CS_1, SPI1_CS_2, SPI1_CS_3, SPI1_MISO, SPI1_MOSI, SPI1_SCK
- net labels removed: +3V3, +BATT, -BATT, CSB0, I2C_SCL, I2C_SDA, MISO, MOSI, NCV0_COM_OUT, SCLK
- wire segments 39 -> 61

Commit message: update parts. add caps
Parts:
- added C1, C2: EEUFR1H151B, CAPPRD500W60D1000H1250, symbol EEUFR1H151B:EEUFR1H151B
- added U10, U6, U8: Small_7_Seg_FlipDot_Module, mio:Small_7_Seg_FlipDot_Module, symbol mio:Small_7_Seg_FlipDot_Module
- added U5, U7, U9: NCV7719, mio:SSOP-24_6.4x7.55mm_P0.65mm, symbol mio:NCV7719
- U1: renamed from U?; footprint (none) -> mio:NUCLEO-F303K8-HEADER
- U2: renamed from U?; footprint (none) -> mio:SLC03B-05
- U3: renamed from U?; symbol flip_dot_clock-rescue:NCV7719-mio -> mio:NCV7719
- U4: renamed from U?; footprint (none) -> mio:Small_7_Seg_FlipDot_Module
Connections:
- net SPI1_CS_0 is gone; now on net SPI1_CS_1: U1.6 (PB0), U3.19 (CSB)
- net +24V: now also C1.P, C2.P, U5.16 (VS2), U5.21 (VS1), U7.16 (VS2), U7.21 (VS1), U9.16 (VS2), U9.21 (VS1)
- net +5V: now also U5.6 (VCC), U7.6 (VCC), U9.6 (VCC)
- net A_SET_1: now also U3.22 (OUT8); no longer U3.2 (OUT1)
- net C_SET_1: now also U3.2 (OUT1); no longer U3.14 (OUT3)
- net D_SET_1: now also U3.3 (OUT5); no longer U3.11 (OUT4)
- net E_SET_1: now also U3.4 (OUT7); no longer U3.3 (OUT5)
- net GND: now also C1.N, C2.N, U5.1 (GND), U5.12 (GND), U5.13 (GND), U5.24 (GND), U7.1 (GND), U7.12 (GND), U7.13 (GND), U7.24 (GND), U9.1 (GND), U9.12 (GND), U9.13 (GND), U9.24 (GND)
- net G_SET_1: now also U3.11 (OUT4); no longer U3.4 (OUT7)
- net RESET_1: now also U3.14 (OUT3); no longer U3.22 (OUT8)
- net SPI1_CS_1: no longer U1.7 (PB7)
- net SPI1_CS_2: now also U1.7 (PB7), U5.19 (CSB); no longer U1.8 (PB6)
- net SPI1_CS_3: now also U1.8 (PB6), U7.19 (CSB); no longer U1.9 (PB1)
- net SPI1_MISO: now also U5.7 (SO), U7.7 (SO), U9.7 (SO)
- net SPI1_MOSI: now also U5.5 (SI), U7.5 (SI), U9.5 (SI)
- net SPI1_SCK: now also U5.20 (SCLK), U7.20 (SCLK), U9.20 (SCLK)
- net NCV_EN_1: now reaches U1.11 (PF1)
- net NCV_EN_1: now also U3.8 (EN)
- net NCV_EN_2: now reaches U1.12 (PA8)
- net NCV_EN_2: now also U5.8 (EN)
- net NCV_EN_3: now reaches U1.13 (PA11)
- net NCV_EN_3: now also U7.8 (EN)
- net NCV_EN_4: now reaches U1.14 (PB5)
- net NCV_EN_4: now also U9.8 (EN)
- net NCV_EN: no longer names the net of U1.24 (PA4)
- net NCV_EN: no longer U3.8 (EN)
- new net A_SET_2: U5.22 (OUT8), U6.1 (A_SET)
- new net A_SET_3: U7.2 (OUT1), U8.1 (A_SET)
- new net A_SET_4: U10.1 (A_SET), U9.2 (OUT1)
- new net B_SET_2: U5.23 (OUT2), U6.2 (B_SET)
- new net B_SET_3: U7.23 (OUT2), U8.2 (B_SET)
- new net B_SET_4: U10.2 (B_SET), U9.23 (OUT2)
- new net C_SET_2: U5.2 (OUT1), U6.3 (C_SET)
- new net C_SET_3: U7.14 (OUT3), U8.3 (C_SET)
- new net C_SET_4: U10.3 (C_SET), U9.14 (OUT3)
- new net D_SET_2: U5.3 (OUT5), U6.4 (D_SET)
- new net D_SET_3: U7.11 (OUT4), U8.4 (D_SET)
- new net D_SET_4: U10.4 (D_SET), U9.11 (OUT4)
- new net E_SET_2: U5.4 (OUT7), U6.5 (E_SET)
- new net E_SET_3: U7.3 (OUT5), U8.5 (E_SET)
- new net E_SET_4: U10.5 (E_SET), U9.3 (OUT5)
- new net F_SET_2: U5.10 (OUT6), U6.6 (F_SET)
- new net F_SET_3: U7.10 (OUT6), U8.6 (F_SET)
- new net F_SET_4: U10.6 (F_SET), U9.10 (OUT6)
- new net G_SET_2: U5.11 (OUT4), U6.7 (G_SET)
- new net G_SET_3: U7.4 (OUT7), U8.7 (G_SET)
- new net G_SET_4: U10.7 (G_SET), U9.4 (OUT7)
- new net RESET_2: U5.14 (OUT3), U6.10 (C_RESET), U6.11 (D_RESET), U6.12 (E_RESET), U6.13 (F_RESET), U6.14 (G_RESET), U6.8 (A_RESET), U6.9 (B_RESET)
- new net RESET_3: U7.22 (OUT8), U8.10 (C_RESET), U8.11 (D_RESET), U8.12 (E_RESET), U8.13 (F_RESET), U8.14 (G_RESET), U8.8 (A_RESET), U8.9 (B_RESET)
- new net RESET_4: U10.10 (C_RESET), U10.11 (D_RESET), U10.12 (E_RESET), U10.13 (F_RESET), U10.14 (G_RESET), U10.8 (A_RESET), U10.9 (B_RESET), U9.22 (OUT8)
- new net SPI1_CS_4: U1.9 (PB1), U9.19 (CSB)
Other:
- moved on the sheet: U1, U2, U3, U4

Commit message: update parts
Parts:
- removed C1, C2: EEUFR1H151B, CAPPRD500W60D1000H1250, symbol EEUFR1H151B:EEUFR1H151B
- added C1: 150uF, Capacitor_THT:CP_Radial_D10.0mm_P5.00mm, symbol Device:CP1
- added C2: 10uF, Capacitor_SMD:C_1206_3216Metric, symbol Device:C
- added C3: 1uF, Capacitor_SMD:C_1206_3216Metric, symbol Device:C
- added C4: 0.1uF, Capacitor_SMD:C_1206_3216Metric, symbol Device:C
- added C5: 10uF, symbol Device:C
- added D1: MRA4003T3G, Diode_SMD:D_SMA, symbol Diode:MRA4003T3G
Connections:
- net +24V: now also C1.1, C2.2, C3.2, C4.2, D1.2 (A); no longer U3.16 (VS2), U3.21 (VS1)
- net +5V: now also C5.1
- net GND: now also C1.2, C2.1, C3.1, C4.1, C5.2
- new net: D1.1 (K), U3.16 (VS2), U3.21 (VS1)
Other:
- moved on the sheet: U3, U4, U5
