File: kicad/control/flip_dot_clock.kicad_pcb (KiCad board)
At the start: 4 copper layers, 126.7 x 38.1 mm, 34 parts, among them J1 Conn_01x02_Male, U1 NUCLEO-F303K8-HEADER, U10 Small_7_Seg_FlipDot_Module, U2 SLC03B-05, U3 NCV7719, U4 Small_7_Seg_FlipDot_Module, U5 NCV7719, U6 Small_7_Seg_FlipDot_Module, U7 NCV7719, U8 Small_7_Seg_FlipDot_Module, U9 NCV7719

Commit message: update
Routing:
- net /SPI1_CS_1: track 86.7 -> 83.2 mm
- net /NCV_EN_1: track 99.4 -> 101.7 mm
- net /SPI1_CS_2: track 62.2 -> 60.4 mm
Changed lines of the file:
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@@
   (via (at 134.493 94.488) (size 0.6) (drill 0.3) (layers "F.Cu" "B.Cu") (net 16))
   (via (at 134.493 97.282) (size 0.6) (drill 0.3) (layers "F.Cu" "B.Cu") (net 16))
+  (segment (start 135.509 93.472) (end 169.545 93.472) (width 0.2) (layer "In1.Cu") (net 16))
+  (segment (start 133.223 98.552) (end 134.493 97.282) (width 0.2) (layer "In1.Cu") (net 16))
   (segment (start 134.493 94.488) (end 135.509 93.472) (width 0.2) (layer "In1.Cu") (net 16))
-  (segment (start 133.223 98.552) (end 134.493 97.282) (width 0.2) (layer "In1.Cu") (net 16))
-  (segment (start 173.482 92.583) (end 173.736 92.329) (width 0.2) (layer "In1.Cu") (net 16))
   (segment (start 121.412 98.552) (end 133.223 98.552) (width 0.2) (layer "In1.Cu") (net 16))
-  (segment (start 173.736 92.329) (end 173.736 89.154) (width 0.2) (layer "In1.Cu") (net 16))
-  (segment (start 172.593 93.472) (end 173.482 92.583) (width 0.2) (layer "In1.Cu") (net 16))
-  (segment (start 135.509 93.472) (end 138.049 93.472) (width 0.2) (layer "In1.Cu") (net 16))
-  (segment (start 138.049 93.472) (end 172.593 93.472) (width 0.2) (layer "In1.Cu") (net 16))
+  (segment (start 171.831 91.186) (end 171.831 88.392) (width 0.2) (layer "In1.Cu") (net 16))
+  (segment (start 169.545 93.472) (end 171.831 91.186) (width 0.2) (layer "In1.Cu") (net 16))
   (segment (start 134.493 97.282) (end 134.493 94.488) (width 0.2) (layer "In2.Cu") (net 16))
   (segment (start 91.7155 98.608) (end 92.639 98.608) (width 0.2) (layer "F.Cu") (net 17))
@@
   (via (at 106.68 97.282) (size 0.6) (drill 0.3) (layers "F.Cu" "B.Cu") (net 17))
   (via (at 94.107 98.552) (size 0.6) (drill 0.3) (layers "F.Cu" "B.Cu") (net 17))
-  (segment (start 170.688 92.71) (end 171.704 91.694) (width 0.2) (layer "In1.Cu") (net 17))
-  (segment (start 106.68 94.488) (end 107.569 93.599) (width 0.2) (layer "In1.Cu") (net 17))
-  (segment (start 117.602 93.599) (end 118.491 92.71) (width 0.2) (layer "In1.Cu") (net 17))
-  (segment (start 107.569 93.599) (end 117.602 93.599) (width 0.2) (layer "In1.Cu") (net 17))
-  (segment (start 118.491 92.71) (end 170.688 92.71) (width 0.2) (layer "In1.Cu") (net 17))
   (segment (start 94.107 98.552) (end 105.41 98.552) (width 0.2) (layer "In1.Cu") (net 17))
-  (segment (start 171.704 91.694) (end 171.704 89.535) (width 0.2) (layer "In1.Cu") (net 17))
+  (segment (start 106.68 94.488) (end 116.84 84.328) (width 0.2) (layer "In1.Cu") (net 17))
+  (segment (start 116.84 84.328) (end 167.259 84.328) (width 0.2) (layer "In1.Cu") (net 17))
   (segment (start 105.41 98.552) (end 106.68 97.282) (width 0.2) (layer "In1.Cu") (net 17))
   (segment (start 106.68 97.282) (end 106.68 94.488) (width 0.2) (layer "In2.Cu") (net 17))
@@
   (segment (start 86.4655 99.908) (end 85.131 99.908) (width 0.2) (layer "F.Cu") (net 57))
   (via (at 85.131 99.908) (size 0.6) (drill 0.3) (layers "F.Cu" "B.Cu") (net 57))
-  (segment (start 103.886 93.853) (end 104.775 93.853) (width 0.2) (layer "In1.Cu") (net 57))
-  (segment (start 104.775 93.853) (end 109.093 89.535) (width 0.2) (layer "In1.Cu") (net 57))
   (segment (start 85.131 99.908) (end 84.455 100.584) (width 0.2) (layer "In1.Cu") (net 57))
-  (segment (start 109.093 89.535) (end 109.982 88.646) (width 0.2) (layer "In1.Cu") (net 57))
-  (segment (start 84.709 93.853) (end 103.886 93.853) (width 0.2) (layer "In1.Cu") (net 57))
+  (segment (start 81.661 93.345) (end 92.456 82.55) (width 0.2) (layer "In1.Cu") (net 57))
   (segment (start 82.677 100.584) (end 81.661 99.568) (width 0.2) (layer "In1.Cu") (net 57))
-  (segment (start 81.661 96.901) (end 84.709 93.853) (width 0.2) (layer "In1.Cu") (net 57))
-  (segment (start 81.661 99.568) (end 81.661 97.917) (width 0.2) (layer "In1.Cu") (net 57))
-  (segment (start 109.982 88.646) (end 168.021 88.646) (width 0.2) (layer "In1.Cu") (net 57))
-  (segment (start 168.021 88.646) (end 169.037 87.63) (width 0.2) (layer "In1.Cu") (net 57))
-  (segment (start 81.661 97.917) (end 81.661 96.901) (width 0.2) (layer "In1.Cu") (net 57))
+  (segment (start 81.661 99.568) (end 81.661 93.345) (width 0.2) (layer "In1.Cu") (net 57))
+  (segment (start 92.456 82.55) (end 167.132 82.55) (width 0.2) (layer "In1.Cu") (net 57))
   (segment (start 84.455 100.584) (end 82.677 100.584) (width 0.2) (layer "In1.Cu") (net 57))
   (segment (start 184.785 98.679) (end 186.055 98.679) (width 0.2) (layer "F.Cu") (net 58))
@@
       (pts
         (xy 205.486 80.899)
-        (xy 205.486 94.615)
-        (xy 176.276 94.615)
-        (xy 176.276 99.441)
-        (xy 169.164 99.441)
-        (xy 169.164 94.996)
-        (xy 150.876 94.996)
-        (xy 150.876 99.441)
-        (xy 131.699 99.441)
-        (xy 131.699 94.996)
-        (xy 113.411 94.996)
-        (xy 113.411 99.441)
-        (xy 104.394 99.441)
-        (xy 104.394 94.996)
-        (xy 86.106 94.996)
-        (xy 86.106 99.441)
-        (xy 79.756 99.441)
+        (xy 205.486 91.694)
+        (xy 196.469 91.694)
+        (xy 196.469 89.281)
+        (xy 178.181 89.281)
+        (xy 178.181 100.965)
+        (xy 169.164 100.965)
+        (xy 169.164 89.281)
+        (xy 150.876 89.281)
+        (xy 150.876 100.965)
+        (xy 131.699 100.965)
+        (xy 131.699 89.281)
+        (xy 113.411 89.281)
+        (xy 113.411 100.965)
+        (xy 104.394 100.965)
+        (xy 104.394 89.281)
+        (xy 86.106 89.281)
+        (xy 86.106 100.965)
+        (xy 79.756 100.965)
         (xy 79.756 80.899)
       )
@@
         (xy 205.486 117.983)
         (xy 79.756 117.983)
-        (xy 79.756 100.076)
-        (xy 86.741 100.076)
-        (xy 86.741 95.631)
-        (xy 103.759 95.631)
-        (xy 103.759 100.076)
-        (xy 114.046 100.076)
-        (xy 114.046 95.631)
-        (xy 131.064 95.631)
-        (xy 131.064 100.076)
-        (xy 151.511 100.076)
-        (xy 151.511 95.631)
-        (xy 168.529 95.631)
-        (xy 168.529 100.076)
-        (xy 176.911 100.076)
-        (xy 176.911 95.25)
-        (xy 205.486 95.25)
+        (xy 79.756 101.6)
+        (xy 86.741 101.6)
+        (xy 86.741 92.329)
+        (xy 103.759 92.329)
+        (xy 103.759 101.6)
+        (xy 114.046 101.6)
+        (xy 114.046 92.329)
+        (xy 131.064 92.329)
+        (xy 131.064 101.6)
+        (xy 151.511 101.6)
+        (xy 151.511 92.329)
+        (xy 168.529 92.329)
+        (xy 168.529 101.6)
+        (xy 178.816 101.6)
+        (xy 178.816 92.329)
+        (xy 205.486 92.329)
       )
     )

Commit message: fix all the kicad files
Parts:
- added J2: Conn_01x15_Female, Connector_PinHeader_2.54mm:PinHeader_1x15_P2.54mm_Vertical, B.Cu at (156.7, 85.3)
- moved U1 30.1 mm to (199.6, 76.6)
Routing:
- net /SPI1_MISO: track 131.6 -> 146.0 mm
- net /NCV_EN_4: track 30.8 -> 43.8 mm
- net /NCV_EN_3: track 68.7 -> 78.6 mm
- net /SPI1_SCK: track 116.2 -> 124.6 mm
- net /SPI1_CS_4: track 16.1 -> 22.6 mm
- net /NCV_EN_2: track 110.3 -> 116.8 mm
- net /SPI1_MOSI: track 115.1 -> 120.6 mm
- net /NCV_EN_1: track 101.7 -> 97.9 mm
- net /SPI1_CS_2: track 60.4 -> 63.3 mm
- net /SPI1_CS_3: track 26.7 -> 28.4 mm
- net /SPI1_CS_1: track 83.2 -> 82.3 mm

Commit message: update pcb
Parts:
- added J3: Conn_01x05_Male, Connector_Molex:Molex_Nano-Fit_105309-xx05_1x05_P2.50mm_Vertical, B.Cu at (113.8, 83.7)
- J2: value Conn_01x15_Female -> Conn_02x08_Odd_Even; footprint Connector_PinHeader_2.54mm:PinHeader_1x15_P2.54mm_Vertical -> Connector_PinSocket_2.54mm:PinSocket_2x10_P2.54mm_Vertical
- moved U1 20.8 mm to (197.7, 55.9)
- moved J2 8.11 mm to (164.8, 86.2)
Connections:
- J2 pad 1: unconnected-(J2-Pin_1) -> /HOUR_DOWN
- J2 pad 10: +5V -> GND
- J2 pad 11: GND -> /SPI1_CS_3
- J2 pad 12: /SPI1_MISO -> unconnected-(J2-Pin_12)
- J2 pad 13: /NCV_EN_4 -> /SPI1_MOSI
- J2 pad 14: /NCV_EN_3 -> unconnected-(J2-Pin_14)
- J2 pad 15: /NCV_EN_2 -> /SPI1_SCK
- J2 pad 2: unconnected-(J2-Pin_2) -> /HOUR_UP
- J2 pad 3: /NCV_EN_1 -> /MIN_UP
- J2 pad 4: /SPI1_CS_1 -> /MIN_DOWN
- J2 pad 5: /SPI1_CS_2 -> /NCV_EN_1
- J2 pad 6: /SPI1_CS_3 -> unconnected-(J2-Pin_6)
- J2 pad 7: /SPI1_MOSI -> /SPI1_CS_1
- J2 pad 8: /SPI1_SCK -> +5V
- J2 pad 9: /SPI1_CS_4 -> /SPI1_CS_2
- U1 pad 1: unconnected-(U1-PA9) -> /HOUR_UP
- U1 pad 15: unconnected-(U1-PB4) -> /MIN_DOWN
- U1 pad 2: unconnected-(U1-PA10) -> /HOUR_DOWN
- U1 pad 5: unconnected-(U1-PA12) -> /MIN_UP
Routing:
- net /MIN_UP: track 0.00 -> 64.5 mm
- net /MIN_DOWN: track 0.00 -> 63.3 mm
- net /HOUR_DOWN: track 0.00 -> 55.9 mm
- net /HOUR_UP: track 0.00 -> 53.4 mm
- net /NCV_EN_2: track 116.8 -> 128.5 mm
- net /NCV_EN_1: track 97.9 -> 105.8 mm
- net /SPI1_CS_1: track 82.3 -> 90.0 mm
- net /NCV_EN_3: track 78.6 -> 84.9 mm
- net /SPI1_MISO: track 146.0 -> 141.2 mm
- net /SPI1_CS_4: track 22.6 -> 26.7 mm
- net /SPI1_SCK: track 124.6 -> 128.0 mm
- net /SPI1_MOSI: track 120.6 -> 123.1 mm
- net /SPI1_CS_3: track 28.4 -> 29.6 mm
- net /NCV_EN_4: track 43.8 -> 43.1 mm

Commit message: moving along
Parts:
- removed C17: 10uF, Capacitor_SMD:C_1206_3216Metric
- removed JP1, JP2: SJ2O, Jumper:SolderJumper-2_P1.3mm_Open_TrianglePad1.0x1.5mm
- removed U1: NUCLEO-F303K8-HEADER, mio:NUCLEO-F303K8-HEADER
- moved J2 3.83 mm to (161.0, 86.2)
Connections:
- J2 pad 12: unconnected-(J2-Pin_12) -> GND
- J2 pad 6: unconnected-(J2-Pin_6) -> +5V
Routing:
- net /SPI1_SCK: track 128.0 -> 121.9 mm
- net /NCV_EN_2: track 128.5 -> 134.0 mm
- net /SPI1_MOSI: track 123.1 -> 118.0 mm
- net /NCV_EN_3: track 84.9 -> 89.7 mm
- net /HOUR_UP: track 53.4 -> 49.1 mm
- net /NCV_EN_4: track 43.1 -> 47.2 mm
- net /MIN_UP: track 64.5 -> 60.5 mm
- net /MIN_DOWN: track 63.3 -> 59.4 mm
- net /SPI1_MISO: track 141.2 -> 145.0 mm
- net /NCV_EN_1: track 105.8 -> 102.2 mm
- net /SPI1_CS_4: track 26.7 -> 23.2 mm
- net /SPI1_CS_1: track 90.0 -> 86.6 mm
- net /HOUR_DOWN: track 55.9 -> 52.6 mm
- net /SPI1_CS_3: track 29.6 -> 27.6 mm
- net /SPI1_CS_2: track 63.4 -> 61.8 mm
- added copper zone on In1.Cu, net +24V
- added copper zone on In1.Cu, net +5V
- removed copper zone on In2.Cu, net +24V
- removed copper zone on In2.Cu, net +5V

Commit message: kicad update
Connections:
- J2 pad 10: GND -> +5V
- J2 pad 14: unconnected-(J2-Pin_14) -> GND
- J2 pad 6: +5V -> unconnected-(J2-Pin_6)

Commit message: add digit holder ground planes
Connections:
- U10 pad 15: unconnected-(U10-NC) -> GND
- U4 pad 15: unconnected-(U4-NC) -> GND
- U6 pad 15: unconnected-(U6-NC) -> GND
- U8 pad 15: unconnected-(U8-NC) -> GND
