File: kicad/control/flip_dot_clock.kicad_sch (KiCad schematic)
At the start: 36 parts, among them J1 Conn_01x02_Male, J2 Conn_02x08_Odd_Even, J3 Conn_01x05_Male, U1 NUCLEO-F303K8-HEADER, U10 Small_7_Seg_FlipDot_Module, U2 SLC03B-05, U3 NCV7719, U4 Small_7_Seg_FlipDot_Module, U5 NCV7719, U6 Small_7_Seg_FlipDot_Module, U7 NCV7719, U8 Small_7_Seg_FlipDot_Module, U9 NCV7719

Commit message: update pcb
Parts:
- added H1, H2, H3, H4, H5, H6: MountingHole, mio:MountingHole_3.2mm_M3, symbol Mechanical:MountingHole
Changed lines of the file:
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@@
     (pin "1")
+  )
+  (symbol (lib_id "Mechanical:MountingHole") (at 46.99 115.57 0) (unit 1)
+    (in_bom yes) (on_board yes) (fields_autoplaced)
+    (property "Reference" "H6" (id 0) (at 49.53 114.935 0)
+      (effects (font (size 1.27 1.27)) (justify left))
+    )
+    (property "Value" "MountingHole" (id 1) (at 49.53 117.475 0)
+      (effects (font (size 1.27 1.27)) (justify left))
+    )
+    (property "Footprint" "mio:MountingHole_3.2mm_M3" (id 2) (at 46.99 115.57 0)
+      (effects (font (size 1.27 1.27)) hide)
+    )
+    (property "Datasheet" "~" (id 3) (at 46.99 115.57 0)
+      (effects (font (size 1.27 1.27)) hide)
+    )
   )
   (symbol (lib_id "power:GND") (at 344.17 201.93 0) (unit 1)
     (in_bom yes) (on_board yes)
-    (property "Reference" "#PWR?" (id 0) (at 344.17 208.28 0)
+    (property "Reference" "#PWR0140" (id 0) (at 344.17 208.28 0)
       (effects (font (size 1.27 1.27)) hide)
     )
@@
     (pin "1")
   )
+  (symbol (lib_id "Mechanical:MountingHole") (at 46.99 100.33 0) (unit 1)
+    (in_bom yes) (on_board yes) (fields_autoplaced)
+    (property "Reference" "H4" (id 0) (at 49.53 99.695 0)
+      (effects (font (size 1.27 1.27)) (justify left))
+    )
+    (property "Value" "MountingHole" (id 1) (at 49.53 102.235 0)
+      (effects (font (size 1.27 1.27)) (justify left))
+    )
+    (property "Footprint" "mio:MountingHole_3.2mm_M3" (id 2) (at 46.99 100.33 0)
+      (effects (font (size 1.27 1.27)) hide)
+    )
+    (property "Datasheet" "~" (id 3) (at 46.99 100.33 0)
+      (effects (font (size 1.27 1.27)) hide)
+    )
+  )
   (symbol (lib_id "power:GND") (at 401.32 160.02 0) (unit 1)
     (in_bom yes) (on_board yes)
@@
     )
     (pin "1")
+  )
+  (symbol (lib_id "Mechanical:MountingHole") (at 46.99 92.71 0) (unit 1)
+    (in_bom yes) (on_board yes) (fields_autoplaced)
+    (property "Reference" "H3" (id 0) (at 49.53 92.075 0)
+      (effects (font (size 1.27 1.27)) (justify left))
+    )
+    (property "Value" "MountingHole" (id 1) (at 49.53 94.615 0)
+      (effects (font (size 1.27 1.27)) (justify left))
+    )
+    (property "Footprint" "mio:MountingHole_3.2mm_M3" (id 2) (at 46.99 92.71 0)
+      (effects (font (size 1.27 1.27)) hide)
+    )
+    (property "Datasheet" "~" (id 3) (at 46.99 92.71 0)
+      (effects (font (size 1.27 1.27)) hide)
+    )
   )
   (symbol (lib_name "NCV7719_1") (lib_id "mio:NCV7719") (at 344.17 78.74 0) (unit 1)
@@
   (symbol (lib_id "power:GND") (at 172.72 99.06 0) (unit 1)
     (in_bom yes) (on_board yes)
-    (property "Reference" "#PWR?" (id 0) (at 172.72 105.41 0)
+    (property "Reference" "#PWR0142" (id 0) (at 172.72 105.41 0)
       (effects (font (size 1.27 1.27)) hide)
     )
@@
     (pin "1")
   )
+  (symbol (lib_id "Mechanical:MountingHole") (at 46.99 77.47 0) (unit 1)
+    (in_bom yes) (on_board yes) (fields_autoplaced)
+    (property "Reference" "H1" (id 0) (at 49.53 76.835 0)
+      (effects (font (size 1.27 1.27)) (justify left))
+    )
+    (property "Value" "MountingHole" (id 1) (at 49.53 79.375 0)
+      (effects (font (size 1.27 1.27)) (justify left))
+    )
+    (property "Footprint" "mio:MountingHole_3.2mm_M3" (id 2) (at 46.99 77.47 0)
+      (effects (font (size 1.27 1.27)) hide)
+    )
+    (property "Datasheet" "~" (id 3) (at 46.99 77.47 0)
+      (effects (font (size 1.27 1.27)) hide)
+    )
+  )
   (symbol (lib_name "NCV7719_3") (lib_id "mio:NCV7719") (at 173.99 180.34 0) (unit 1)
     (in_bom yes) (on_board yes)
@@
   (symbol (lib_id "power:GND") (at 344.17 100.33 0) (unit 1)
     (in_bom yes) (on_board yes)
-    (property "Reference" "#PWR?" (id 0) (at 344.17 106.68 0)
+    (property "Reference" "#PWR0139" (id 0) (at 344.17 106.68 0)
       (effects (font (size 1.27 1.27)) hide)
     )
@@
     (pin "2")
   )
+  (symbol (lib_id "Mechanical:MountingHole") (at 46.99 107.95 0) (unit 1)
+    (in_bom yes) (on_board yes) (fields_autoplaced)
+    (property "Reference" "H5" (id 0) (at 49.53 107.315 0)
+      (effects (font (size 1.27 1.27)) (justify left))
+    )
+    (property "Value" "MountingHole" (id 1) (at 49.53 109.855 0)
+      (effects (font (size 1.27 1.27)) (justify left))
+    )
+    (property "Footprint" "mio:MountingHole_3.2mm_M3" (id 2) (at 46.99 107.95 0)
+      (effects (font (size 1.27 1.27)) hide)
+    )
+    (property "Datasheet" "~" (id 3) (at 46.99 107.95 0)
+      (effects (font (size 1.27 1.27)) hide)
+    )
+  )
   (symbol (lib_id "Device:C") (at 392.43 146.05 270) (unit 1)
     (in_bom yes) (on_board yes)
@@
   (symbol (lib_id "power:GND") (at 173.99 201.93 0) (unit 1)
     (in_bom yes) (on_board yes)
-    (property "Reference" "#PWR?" (id 0) (at 173.99 208.28 0)
+    (property "Reference" "#PWR0141" (id 0) (at 173.99 208.28 0)
       (effects (font (size 1.27 1.27)) hide)
     )
@@
     (pin "2")
   )
+  (symbol (lib_id "Mechanical:MountingHole") (at 46.99 85.09 0) (unit 1)
+    (in_bom yes) (on_board yes) (fields_autoplaced)
+    (property "Reference" "H2" (id 0) (at 49.53 84.455 0)
+      (effects (font (size 1.27 1.27)) (justify left))
+    )
+    (property "Value" "MountingHole" (id 1) (at 49.53 86.995 0)
+      (effects (font (size 1.27 1.27)) (justify left))
+    )
+    (property "Footprint" "mio:MountingHole_3.2mm_M3" (id 2) (at 46.99 85.09 0)
+      (effects (font (size 1.27 1.27)) hide)
+    )
+    (property "Datasheet" "~" (id 3) (at 46.99 85.09 0)
+      (effects (font (size 1.27 1.27)) hide)
+    )
+  )
   (symbol (lib_id "power:GND") (at 255.27 166.37 0) (unit 1)
     (in_bom yes) (on_board yes) (fields_autoplaced)
@@
       (reference "#PWR0138") (unit 1) (value "GND") (footprint "")
     )
+    (path "/8d44a10e-b0c1-4575-a5d4-f2bd81a28341"
+      (reference "#PWR0139") (unit 1) (value "GND") (footprint "")
+    )
     (path "/0b23e1bb-408d-464c-8c81-13e2b5d23e23"
-      (reference "#PWR?") (unit 1) (value "GND") (footprint "")
+      (reference "#PWR0140") (unit 1) (value "GND") (footprint "")
+    )
+    (path "/cd8db88a-a85b-4097-8ce4-a731999d11db"
+      (reference "#PWR0141") (unit 1) (value "GND") (footprint "")
     )
     (path "/5ec3df19-7cf3-459a-8399-72a32e477a5b"
-      (reference "#PWR?") (unit 1) (value "GND") (footprint "")
-    )
-    (path "/8d44a10e-b0c1-4575-a5d4-f2bd81a28341"
-      (reference "#PWR?") (unit 1) (value "GND") (footprint "")
-    )
-    (path "/cd8db88a-a85b-4097-8ce4-a731999d11db"
-      (reference "#PWR?") (unit 1) (value "GND") (footprint "")
+      (reference "#PWR0142") (unit 1) (value "GND") (footprint "")
     )
     (path "/00000000-0000-0000-0000-000061f1c429"
@@
       (reference "D4") (unit 1) (value "MRA4003T3G") (footprint "Diode_SMD:D_SMA")
     )
+    (path "/84625814-3c34-4997-9c1c-566a30048a0f"
+      (reference "H1") (unit 1) (value "MountingHole") (footprint "mio:MountingHole_3.2mm_M3")
+    )
+    (path "/e476f79c-e0c8-465e-9770-99d67609efe1"
+      (reference "H2") (unit 1) (value "MountingHole") (footprint "mio:MountingHole_3.2mm_M3")
+    )
+    (path "/526b57b0-b37b-483d-9fc8-5f845ac22fbb"
+      (reference "H3") (unit 1) (value "MountingHole") (footprint "mio:MountingHole_3.2mm_M3")
+    )
+    (path "/44eb7b55-8f82-421f-960a-57dc31a92d41"
+      (reference "H4") (unit 1) (value "MountingHole") (footprint "mio:MountingHole_3.2mm_M3")
+    )
+    (path "/ab1b7d11-55e5-4e38-9613-3879ddaad3e5"
+      (reference "H5") (unit 1) (value "MountingHole") (footprint "mio:MountingHole_3.2mm_M3")
+    )
+    (path "/0295d699-0dd3-436d-ac96-acc871b2e66d"
+      (reference "H6") (unit 1) (value "MountingHole") (footprint "mio:MountingHole_3.2mm_M3")
+    )
     (path "/d170073c-990e-452b-9e72-8bd3cb8f7a66"
