File: kicad/control/flip_dot_clock.kicad_sch (KiCad schematic)
At the start: 42 parts, among them J1 Conn_01x02_Male, J2 Conn_02x08_Odd_Even, J3 Conn_01x05_Male, U1 NUCLEO-F303K8-HEADER, U10 Small_7_Seg_FlipDot_Module, U2 SLC03B-05, U3 NCV7719, U4 Small_7_Seg_FlipDot_Module, U5 NCV7719, U6 Small_7_Seg_FlipDot_Module, U7 NCV7719, U8 Small_7_Seg_FlipDot_Module, U9 NCV7719

Commit message: update
Connections:
- net HOUR_DOWN: now also J2.2 (Pin_2), J3.1 (Pin_1), U1.1 (PA9); no longer J2.1 (Pin_1), J3.2 (Pin_2), U1.5 (PA12)
- net HOUR_UP: now also J2.1 (Pin_1), J3.2 (Pin_2), U1.5 (PA12); no longer J2.2 (Pin_2), J3.1 (Pin_1), U1.1 (PA9)
- net MIN_DOWN: now also J2.3 (Pin_3), J3.3 (Pin_3), U1.6 (PB0); no longer J2.4 (Pin_4), J3.4 (Pin_4), U1.2 (PA10)
- net MIN_UP: now also J2.4 (Pin_4), J3.4 (Pin_4), U1.2 (PA10); no longer J2.3 (Pin_3), J3.3 (Pin_3), U1.6 (PB0)
Changed lines of the file:
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@@
-(kicad_sch (version 20220328) (generator eeschema)
+(kicad_sch (version 20220331) (generator eeschema)
   (paper "A3")
   (junction (at 135.89 76.2) (diameter 0) (color 0 0 0 0)
@@
     (effects (font (size 1.27 1.27)) (justify right bottom))
   )
-  (label "MIN_DOWN" (at 83.82 222.25 0) (fields_autoplaced)
+  (label "MIN_UP" (at 83.82 222.25 0) (fields_autoplaced)
     (effects (font (size 1.27 1.27)) (justify right bottom))
   )
@@
     (effects (font (size 1.27 1.27)) (justify right bottom))
   )
-  (label "MIN_UP" (at 171.45 228.6 0) (fields_autoplaced)
+  (label "MIN_DOWN" (at 171.45 228.6 0) (fields_autoplaced)
     (effects (font (size 1.27 1.27)) (justify right bottom))
   )
@@
     (effects (font (size 1.27 1.27)) (justify left bottom))
   )
-  (label "MIN_UP" (at 290.83 229.87 0) (fields_autoplaced)
-    (effects (font (size 1.27 1.27)) (justify left bottom))
-  )
-  (label "HOUR_DOWN" (at 290.83 227.33 0) (fields_autoplaced)
+  (label "MIN_DOWN" (at 290.83 229.87 0) (fields_autoplaced)
+    (effects (font (size 1.27 1.27)) (justify left bottom))
+  )
+  (label "HOUR_UP" (at 290.83 227.33 0) (fields_autoplaced)
     (effects (font (size 1.27 1.27)) (justify left bottom))
   )
@@
     (effects (font (size 1.27 1.27)) (justify right bottom))
   )
-  (label "HOUR_UP" (at 83.82 218.44 0) (fields_autoplaced)
+  (label "HOUR_DOWN" (at 83.82 218.44 0) (fields_autoplaced)
     (effects (font (size 1.27 1.27)) (justify right bottom))
   )
@@
     (effects (font (size 1.27 1.27)) (justify right bottom))
   )
-  (label "HOUR_DOWN" (at 171.45 226.06 0) (fields_autoplaced)
+  (label "HOUR_UP" (at 171.45 226.06 0) (fields_autoplaced)
     (effects (font (size 1.27 1.27)) (justify right bottom))
   )
@@
     (effects (font (size 1.27 1.27)) (justify left bottom))
   )
-  (label "MIN_DOWN" (at 196.85 228.6 0) (fields_autoplaced)
+  (label "MIN_UP" (at 196.85 228.6 0) (fields_autoplaced)
     (effects (font (size 1.27 1.27)) (justify left bottom))
   )
@@
     (effects (font (size 1.27 1.27)) (justify left bottom))
   )
-  (label "MIN_DOWN" (at 290.83 232.41 0) (fields_autoplaced)
+  (label "MIN_UP" (at 290.83 232.41 0) (fields_autoplaced)
     (effects (font (size 1.27 1.27)) (justify left bottom))
   )
@@
     (effects (font (size 1.27 1.27)) (justify right bottom))
   )
-  (label "MIN_UP" (at 83.82 237.49 0) (fields_autoplaced)
+  (label "MIN_DOWN" (at 83.82 237.49 0) (fields_autoplaced)
     (effects (font (size 1.27 1.27)) (justify right bottom))
   )
@@
     (effects (font (size 1.27 1.27)) (justify left bottom))
   )
-  (label "HOUR_UP" (at 290.83 224.79 0) (fields_autoplaced)
+  (label "HOUR_DOWN" (at 290.83 224.79 0) (fields_autoplaced)
     (effects (font (size 1.27 1.27)) (justify left bottom))
   )
@@
     (effects (font (size 1.27 1.27)) (justify right bottom))
   )
-  (label "HOUR_UP" (at 196.85 226.06 0) (fields_autoplaced)
+  (label "HOUR_DOWN" (at 196.85 226.06 0) (fields_autoplaced)
     (effects (font (size 1.27 1.27)) (justify left bottom))
   )
@@
     (effects (font (size 1.27 1.27)) (justify left bottom))
   )
-  (label "HOUR_DOWN" (at 83.82 233.68 0) (fields_autoplaced)
-    (effects (font (size 1.27 1.27)) (justify right bottom))
-  )
+  (label "HOUR_UP" (at 83.82 233.68 0) (fields_autoplaced)
+    (effects (font (size 1.27 1.27)) (justify right bottom))
+  )
