File: kicad/button_board/button_board.kicad_sch (KiCad schematic)
At the start: 9 parts, among them J1 Conn_01x05_Male, SW1 apem-3eth9-15.0, SW2 apem-3eth9-15.0, SW3 apem-3eth9-15.0, SW4 apem-3eth9-15.0

Commit message: update
Connections:
- net HOUR_DOWN: now also J1.1 (Pin_1), SW1.1, SW1.2; no longer J1.2 (Pin_2), SW2.1, SW2.2
- net HOUR_UP: now also J1.2 (Pin_2), SW2.1, SW2.2; no longer J1.1 (Pin_1), SW1.1, SW1.2
- net MIN_DOWN: now also J1.3 (Pin_3), SW3.1, SW3.2; no longer J1.4 (Pin_4), SW4.1, SW4.2
- net MIN_UP: now also J1.4 (Pin_4), SW4.1, SW4.2; no longer J1.3 (Pin_3), SW3.1, SW3.2
Changed lines of the file:
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@@
-(kicad_sch (version 20220126) (generator eeschema)
+(kicad_sch (version 20220331) (generator eeschema)
   (paper "A4")
   (junction (at 109.22 72.39) (diameter 0) (color 0 0 0 0)
@@
     (stroke (width 0) (type default))
   )
-  (label "MIN_DOWN" (at 203.2 88.9 0) (fields_autoplaced)
+  (label "MIN_UP" (at 203.2 88.9 0) (fields_autoplaced)
     (effects (font (size 1.27 1.27)) (justify left bottom))
   )
-  (label "HOUR_DOWN" (at 203.2 83.82 0) (fields_autoplaced)
+  (label "HOUR_UP" (at 203.2 83.82 0) (fields_autoplaced)
     (effects (font (size 1.27 1.27)) (justify left bottom))
   )
-  (label "MIN_UP" (at 203.2 86.36 0) (fields_autoplaced)
+  (label "MIN_DOWN" (at 203.2 86.36 0) (fields_autoplaced)
     (effects (font (size 1.27 1.27)) (justify left bottom))
   )
-  (label "MIN_DOWN" (at 158.75 97.79 0) (fields_autoplaced)
+  (label "MIN_UP" (at 158.75 97.79 0) (fields_autoplaced)
     (effects (font (size 1.27 1.27)) (justify left bottom))
   )
-  (label "MIN_UP" (at 160.02 72.39 0) (fields_autoplaced)
+  (label "MIN_DOWN" (at 160.02 72.39 0) (fields_autoplaced)
     (effects (font (size 1.27 1.27)) (justify left bottom))
   )
-  (label "HOUR_UP" (at 203.2 81.28 0) (fields_autoplaced)
+  (label "HOUR_DOWN" (at 203.2 81.28 0) (fields_autoplaced)
     (effects (font (size 1.27 1.27)) (justify left bottom))
   )
-  (label "HOUR_UP" (at 113.03 72.39 0) (fields_autoplaced)
+  (label "HOUR_DOWN" (at 113.03 72.39 0) (fields_autoplaced)
     (effects (font (size 1.27 1.27)) (justify left bottom))
   )
-  (label "HOUR_DOWN" (at 111.76 97.79 0) (fields_autoplaced)
+  (label "HOUR_UP" (at 111.76 97.79 0) (fields_autoplaced)
     (effects (font (size 1.27 1.27)) (justify left bottom))
   )
