File: kicad/nucleo_interposer/nucleo_interposer.kicad_pcb (KiCad board)
At the start: 2 copper layers, 20.3 x 70.9 mm, 7 parts, among them J1 Conn_02x08_Odd_Even, U1 NUCLEO-F303K8-HEADER

Commit message: update
Connections:
- J1 pad 1: /HOUR_DOWN -> /HOUR_UP
- J1 pad 2: /HOUR_UP -> /HOUR_DOWN
- J1 pad 3: /MIN_UP -> /MIN_DOWN
- J1 pad 4: /MIN_DOWN -> /MIN_UP
- U1 pad 1: /HOUR_UP -> /HOUR_DOWN
- U1 pad 2: /MIN_DOWN -> /MIN_UP
- U1 pad 5: /HOUR_DOWN -> /HOUR_UP
- U1 pad 6: /MIN_UP -> /MIN_DOWN
Routing:
- net /MIN_UP: track 11.8 -> 7.61 mm
- net /MIN_DOWN: track 7.61 -> 11.8 mm
- net /HOUR_UP: track 7.61 -> 11.4 mm
- net /HOUR_DOWN: track 11.4 -> 7.61 mm
Changed lines of the file:
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@@
-(kicad_pcb (version 20220308) (generator pcbnew)
+(kicad_pcb (version 20220331) (generator pcbnew)
   (general
     (thickness 1.6)
@@
     (pcbplotparams
       (layerselection 0x00010fc_ffffffff)
+      (plot_on_all_layers_selection 0x0000000_00000000)
       (disableapertmacros false)
       (usegerberextensions true)
@@
       (dashed_line_gap_ratio 3.000000)
       (svgprecision 4)
-      (excludeedgelayer true)
       (plotframeref false)
       (viasonmask false)
@@
     (property "Sheetfile" "nucleo_interposer.kicad_sch")
     (property "Sheetname" "")
+    (property "ki_description" "Mounting Hole without connection")
+    (property "ki_keywords" "mounting hole")
     (clearance 0.508)
     (attr exclude_from_pos_files)
@@
       (stroke (width 0.12) (type solid)) (layer "User.1"))
     (pad "1" thru_hole rect (at 1.675 -41.6) (size 1.7 1.7) (drill 1) (layers *.Cu *.Mask)
-      (net 4 "/HOUR_UP") (pinfunction "PA9") (pintype "bidirectional"))
+      (net 3 "/HOUR_DOWN") (pinfunction "PA9") (pintype "bidirectional"))
     (pad "2" thru_hole circle (at 1.675 -39.06) (size 1.7 1.7) (drill 1) (layers *.Cu *.Mask)
-      (net 6 "/MIN_DOWN") (pinfunction "PA10") (pintype "bidirectional"))
+      (net 5 "/MIN_UP") (pinfunction "PA10") (pintype "bidirectional"))
     (pad "3" thru_hole circle (at 1.675 -36.52) (size 1.7 1.7) (drill 1) (layers *.Cu *.Mask)
       (net 21 "unconnected-(U1-NRST)") (pinfunction "NRST") (pintype "no_connect"))
@@
       (net 1 "GND") (pinfunction "GND") (pintype "bidirectional"))
     (pad "5" thru_hole circle (at 1.675 -31.44) (size 1.7 1.7) (drill 1) (layers *.Cu *.Mask)
-      (net 3 "/HOUR_DOWN") (pinfunction "PA12") (pintype "bidirectional"))
+      (net 4 "/HOUR_UP") (pinfunction "PA12") (pintype "bidirectional"))
     (pad "6" thru_hole circle (at 1.675 -28.9) (size 1.7 1.7) (drill 1) (layers *.Cu *.Mask)
-      (net 5 "/MIN_UP") (pinfunction "PB0") (pintype "bidirectional"))
+      (net 6 "/MIN_DOWN") (pinfunction "PB0") (pintype "bidirectional"))
     (pad "7" thru_hole circle (at 1.675 -26.36) (size 1.7 1.7) (drill 1) (layers *.Cu *.Mask)
       (net 7 "/NCV_EN_1") (pinfunction "PB7") (pintype "bidirectional"))
@@
     (property "Sheetfile" "nucleo_interposer.kicad_sch")
     (property "Sheetname" "")
+    (property "ki_description" "Mounting Hole without connection")
+    (property "ki_keywords" "mounting hole")
     (clearance 0.508)
     (attr exclude_from_pos_files)
@@
     (property "Sheetfile" "nucleo_interposer.kicad_sch")
     (property "Sheetname" "")
+    (property "ki_description" "Generic connector, double row, 02x10, odd/even pin numbering scheme (row 1 odd numbers, row 2 even numbers), script generated (kicad-library-utils/schlib/autogen/connector/)")
+    (property "ki_keywords" "connector")
     (attr through_hole)
     (fp_text reference "J1" (at 1.27 2.33) (layer "B.SilkS")
@@
       (stroke (width 0.1) (type solid)) (layer "B.Fab"))
     (pad "1" thru_hole rect (at 0 0 180) (size 1.7 1.7) (drill 1) (layers *.Cu *.Mask)
-      (net 3 "/HOUR_DOWN") (pinfunction "Pin_1") (pintype "passive"))
+      (net 4 "/HOUR_UP") (pinfunction "Pin_1") (pintype "passive"))
     (pad "2" thru_hole oval (at 2.54 0 180) (size 1.7 1.7) (drill 1) (layers *.Cu *.Mask)
-      (net 4 "/HOUR_UP") (pinfunction "Pin_2") (pintype "passive"))
+      (net 3 "/HOUR_DOWN") (pinfunction "Pin_2") (pintype "passive"))
     (pad "3" thru_hole oval (at 0 -2.54 180) (size 1.7 1.7) (drill 1) (layers *.Cu *.Mask)
-      (net 5 "/MIN_UP") (pinfunction "Pin_3") (pintype "passive"))
+      (net 6 "/MIN_DOWN") (pinfunction "Pin_3") (pintype "passive"))
     (pad "4" thru_hole oval (at 2.54 -2.54 180) (size 1.7 1.7) (drill 1) (layers *.Cu *.Mask)
-      (net 6 "/MIN_DOWN") (pinfunction "Pin_4") (pintype "passive"))
+      (net 5 "/MIN_UP") (pinfunction "Pin_4") (pintype "passive"))
     (pad "5" thru_hole oval (at 0 -5.08 180) (size 1.7 1.7) (drill 1) (layers *.Cu *.Mask)
       (net 7 "/NCV_EN_1") (pinfunction "Pin_5") (pintype "passive"))
@@
     (property "Sheetfile" "nucleo_interposer.kicad_sch")
     (property "Sheetname" "")
+    (property "ki_description" "Solder Jumper, 2-pole, open")
+    (property "ki_keywords" "solder jumper SPST")
     (attr exclude_from_pos_files)
     (fp_text reference "JP1" (at -3.2004 0) (layer "B.SilkS")
@@
     (property "Sheetfile" "nucleo_interposer.kicad_sch")
     (property "Sheetname" "")
+    (property "ki_description" "Solder Jumper, 2-pole, open")
+    (property "ki_keywords" "solder jumper SPST")
     (attr exclude_from_pos_files)
     (fp_text reference "JP2" (at -3.2004 0) (layer "B.SilkS")
@@
     (property "Sheetfile" "nucleo_interposer.kicad_sch")
     (property "Sheetname" "")
+    (property "ki_description" "Unpolarized capacitor")
+    (property "ki_keywords" "cap capacitor")
     (attr smd)
     (fp_text reference "C1" (at 3.478 0 90) (layer "B.SilkS")
@@
   (segment (start 148.3512 78.601) (end 148.336 78.5858) (width 0.4) (layer "B.Cu") (net 2))
   (segment (start 144.6414 102.743) (end 146.685 102.743) (width 0.4) (layer "B.Cu") (net 2))
-  (segment (start 143.129 77.216) (end 144.399 75.946) (width 0.2) (layer "F.Cu") (net 3))
-  (segment (start 142.494 79.756) (end 143.129 79.121) (width 0.2) (layer "F.Cu") (net 3))
-  (segment (start 143.129 79.121) (end 143.129 77.216) (width 0.2) (layer "F.Cu") (net 3))
-  (segment (start 137.693 79.756) (end 142.494 79.756) (width 0.2) (layer "F.Cu") (net 3))
-  (segment (start 136.308 81.141) (end 137.693 79.756) (width 0.2) (layer "F.Cu") (net 3))
-  (segment (start 136.894 70.981) (end 136.308 70.981) (width 0.2) (layer "F.Cu") (net 4))
-  (segment (start 141.859 75.946) (end 136.894 70.981) (width 0.2) (layer "F.Cu") (net 4))
-  (segment (start 143.129 79.756) (end 144.399 78.486) (width 0.2) (layer "F.Cu") (net 5))
-  (segment (start 143.129 81.6864) (end 143.129 79.756) (width 0.2) (layer "F.Cu") (net 5))
-  (segment (start 136.308 83.681) (end 137.693 82.296) (width 0.2) (layer "F.Cu") (net 5))
-  (segment (start 137.693 82.296) (end 142.5194 82.296) (width 0.2) (layer "F.Cu") (net 5))
-  (segment (start 142.5194 82.296) (end 143.129 81.6864) (width 0.2) (layer "F.Cu") (net 5))
-  (segment (start 144.4244 78.847805) (end 144.4244 78.4352) (width 0.2) (layer "F.Cu") (net 5))
-  (segment (start 136.894 73.521) (end 136.308 73.521) (width 0.2) (layer "F.Cu") (net 6))
-  (segment (start 141.859 78.486) (end 136.894 73.521) (width 0.2) (layer "F.Cu") (net 6))
+  (segment (start 136.894 70.981) (end 136.308 70.981) (width 0.2) (layer "F.Cu") (net 3))
+  (segment (start 141.859 75.946) (end 136.894 70.981) (width 0.2) (layer "F.Cu") (net 3))
+  (segment (start 143.129 77.216) (end 144.399 75.946) (width 0.2) (layer "F.Cu") (net 4))
+  (segment (start 142.494 79.756) (end 143.129 79.121) (width 0.2) (layer "F.Cu") (net 4))
+  (segment (start 143.129 79.121) (end 143.129 77.216) (width 0.2) (layer "F.Cu") (net 4))
+  (segment (start 137.693 79.756) (end 142.494 79.756) (width 0.2) (layer "F.Cu") (net 4))
+  (segment (start 136.308 81.141) (end 137.693 79.756) (width 0.2) (layer "F.Cu") (net 4))
+  (segment (start 136.894 73.521) (end 136.308 73.521) (width 0.2) (layer "F.Cu") (net 5))
+  (segment (start 141.859 78.486) (end 136.894 73.521) (width 0.2) (layer "F.Cu") (net 5))
+  (segment (start 143.129 79.756) (end 144.399 78.486) (width 0.2) (layer "F.Cu") (net 6))
+  (segment (start 143.129 81.6864) (end 143.129 79.756) (width 0.2) (layer "F.Cu") (net 6))
+  (segment (start 136.308 83.681) (end 137.693 82.296) (width 0.2) (layer "F.Cu") (net 6))
+  (segment (start 137.693 82.296) (end 142.5194 82.296) (width 0.2) (layer "F.Cu") (net 6))
+  (segment (start 142.5194 82.296) (end 143.129 81.6864) (width 0.2) (layer "F.Cu") (net 6))
+  (segment (start 144.4244 78.847805) (end 144.4244 78.4352) (width 0.2) (layer "F.Cu") (net 6))
   (segment (start 136.308 86.221) (end 140.233 82.296) (width 0.2) (layer "B.Cu") (net 7))
   (segment (start 143.129 82.296) (end 144.399 81.026) (width 0.2) (layer "B.Cu") (net 7))
