File: kicad/nucleo_interposer/nucleo_interposer.kicad_sch (KiCad schematic)
At the start: 5 parts, among them J1 Conn_02x08_Odd_Even, U1 NUCLEO-F303K8-HEADER

Commit message: update pcb
Parts:
- added H1, H2: MountingHole, mio:MountingHole_3.2mm_M3, symbol Mechanical:MountingHole
Changed lines of the file:
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@@
     (effects (font (size 1.27 1.27)) (justify left bottom))
+  )
+  (symbol (lib_id "Mechanical:MountingHole") (at 66.04 38.1 0) (unit 1)
+    (in_bom yes) (on_board yes) (fields_autoplaced)
+    (property "Reference" "H2" (id 0) (at 68.58 37.465 0)
+      (effects (font (size 1.27 1.27)) (justify left))
+    )
+    (property "Value" "MountingHole" (id 1) (at 68.58 40.005 0)
+      (effects (font (size 1.27 1.27)) (justify left))
+    )
+    (property "Footprint" "mio:MountingHole_3.2mm_M3" (id 2) (at 66.04 38.1 0)
+      (effects (font (size 1.27 1.27)) hide)
+    )
+    (property "Datasheet" "~" (id 3) (at 66.04 38.1 0)
+      (effects (font (size 1.27 1.27)) hide)
+    )
   )
   (symbol (lib_id "power:GND") (at 223.52 83.82 0) (unit 1)
@@
     (pin "1")
   )
+  (symbol (lib_id "Mechanical:MountingHole") (at 66.04 30.48 0) (unit 1)
+    (in_bom yes) (on_board yes) (fields_autoplaced)
+    (property "Reference" "H1" (id 0) (at 68.58 29.845 0)
+      (effects (font (size 1.27 1.27)) (justify left))
+    )
+    (property "Value" "MountingHole" (id 1) (at 68.58 32.385 0)
+      (effects (font (size 1.27 1.27)) (justify left))
+    )
+    (property "Footprint" "mio:MountingHole_3.2mm_M3" (id 2) (at 66.04 30.48 0)
+      (effects (font (size 1.27 1.27)) hide)
+    )
+    (property "Datasheet" "~" (id 3) (at 66.04 30.48 0)
+      (effects (font (size 1.27 1.27)) hide)
+    )
+  )
   (symbol (lib_name "SolderJumper_2_Open_1") (lib_id "Jumper:SolderJumper_2_Open") (at 78.74 99.06 0) (unit 1)
     (in_bom yes) (on_board yes)
@@
       (reference "C1") (unit 1) (value "C") (footprint "Capacitor_SMD:C_1206_3216Metric")
     )
+    (path "/964bb0ec-e558-45e4-9bb0-7f8e8f3ab707"
+      (reference "H1") (unit 1) (value "MountingHole") (footprint "mio:MountingHole_3.2mm_M3")
+    )
+    (path "/0bfb77c8-e9e0-4927-beab-c0480cf12de8"
+      (reference "H2") (unit 1) (value "MountingHole") (footprint "mio:MountingHole_3.2mm_M3")
+    )
     (path "/ae3fa950-2190-483a-a194-82d75f4839b7"

Commit message: dfm
Parts:
- H1, H2: value MountingHole -> (none); footprint mio:MountingHole_3.2mm_M3 -> (none)
Changed lines of the file:
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@@
       (effects (font (size 1.27 1.27)) (justify left))
     )
-    (property "Value" "MountingHole" (id 1) (at 68.58 40.005 0)
+    (property "Value" "" (id 1) (at 68.58 40.005 0)
       (effects (font (size 1.27 1.27)) (justify left))
     )
-    (property "Footprint" "mio:MountingHole_3.2mm_M3" (id 2) (at 66.04 38.1 0)
+    (property "Footprint" "" (id 2) (at 66.04 38.1 0)
       (effects (font (size 1.27 1.27)) hide)
     )
@@
       (effects (font (size 1.27 1.27)) (justify left))
     )
-    (property "Value" "MountingHole" (id 1) (at 68.58 32.385 0)
+    (property "Value" "" (id 1) (at 68.58 32.385 0)
       (effects (font (size 1.27 1.27)) (justify left))
     )
-    (property "Footprint" "mio:MountingHole_3.2mm_M3" (id 2) (at 66.04 30.48 0)
+    (property "Footprint" "" (id 2) (at 66.04 30.48 0)
       (effects (font (size 1.27 1.27)) hide)
     )

Commit message: update
Parts:
- H1, H2: value (none) -> MountingHole; footprint (none) -> mio:MountingHole_3.2mm_M3
Connections:
- net HOUR_DOWN: now also J1.2 (Pin_2), U1.1 (PA9); no longer J1.1 (Pin_1), U1.5 (PA12)
- net HOUR_UP: now also J1.1 (Pin_1), U1.5 (PA12); no longer J1.2 (Pin_2), U1.1 (PA9)
- net MIN_DOWN: now also J1.3 (Pin_3), U1.6 (PB0); no longer J1.4 (Pin_4), U1.2 (PA10)
- net MIN_UP: now also J1.4 (Pin_4), U1.2 (PA10); no longer J1.3 (Pin_3), U1.6 (PB0)
Changed lines of the file:
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@@
-(kicad_sch (version 20220126) (generator eeschema)
+(kicad_sch (version 20220331) (generator eeschema)
   (paper "A4")
   (junction (at 205.74 78.74) (diameter 0) (color 0 0 0 0)
@@
     (effects (font (size 1.27 1.27)) (justify right bottom))
   )
-  (label "MIN_UP" (at 184.15 71.12 0) (fields_autoplaced)
-    (effects (font (size 1.27 1.27)) (justify right bottom))
-  )
-  (label "HOUR_UP" (at 96.52 60.96 0) (fields_autoplaced)
+  (label "MIN_DOWN" (at 184.15 71.12 0) (fields_autoplaced)
+    (effects (font (size 1.27 1.27)) (justify right bottom))
+  )
+  (label "HOUR_DOWN" (at 96.52 60.96 0) (fields_autoplaced)
     (effects (font (size 1.27 1.27)) (justify right bottom))
   )
@@
     (effects (font (size 1.27 1.27)) (justify left bottom))
   )
-  (label "MIN_DOWN" (at 96.52 64.77 0) (fields_autoplaced)
+  (label "MIN_UP" (at 96.52 64.77 0) (fields_autoplaced)
     (effects (font (size 1.27 1.27)) (justify right bottom))
   )
@@
     (effects (font (size 1.27 1.27)) (justify right bottom))
   )
-  (label "HOUR_UP" (at 209.55 68.58 0) (fields_autoplaced)
+  (label "HOUR_DOWN" (at 209.55 68.58 0) (fields_autoplaced)
     (effects (font (size 1.27 1.27)) (justify left bottom))
   )
@@
     (effects (font (size 1.27 1.27)) (justify left bottom))
   )
-  (label "MIN_DOWN" (at 209.55 71.12 0) (fields_autoplaced)
+  (label "MIN_UP" (at 209.55 71.12 0) (fields_autoplaced)
     (effects (font (size 1.27 1.27)) (justify left bottom))
   )
@@
     (effects (font (size 1.27 1.27)) (justify right bottom))
   )
-  (label "HOUR_DOWN" (at 184.15 68.58 0) (fields_autoplaced)
-    (effects (font (size 1.27 1.27)) (justify right bottom))
-  )
-  (label "MIN_UP" (at 96.52 80.01 0) (fields_autoplaced)
+  (label "HOUR_UP" (at 184.15 68.58 0) (fields_autoplaced)
+    (effects (font (size 1.27 1.27)) (justify right bottom))
+  )
+  (label "MIN_DOWN" (at 96.52 80.01 0) (fields_autoplaced)
     (effects (font (size 1.27 1.27)) (justify right bottom))
   )
@@
     (effects (font (size 1.27 1.27)) (justify left bottom))
   )
-  (label "HOUR_DOWN" (at 96.52 76.2 0) (fields_autoplaced)
+  (label "HOUR_UP" (at 96.52 76.2 0) (fields_autoplaced)
     (effects (font (size 1.27 1.27)) (justify right bottom))
   )
@@
       (effects (font (size 1.27 1.27)) (justify left))
     )
-    (property "Value" "" (id 1) (at 68.58 40.005 0)
+    (property "Value" "MountingHole" (id 1) (at 68.58 40.005 0)
       (effects (font (size 1.27 1.27)) (justify left))
     )
-    (property "Footprint" "" (id 2) (at 66.04 38.1 0)
+    (property "Footprint" "mio:MountingHole_3.2mm_M3" (id 2) (at 66.04 38.1 0)
       (effects (font (size 1.27 1.27)) hide)
     )
@@
       (effects (font (size 1.27 1.27)) (justify left))
     )
-    (property "Value" "" (id 1) (at 68.58 32.385 0)
+    (property "Value" "MountingHole" (id 1) (at 68.58 32.385 0)
       (effects (font (size 1.27 1.27)) (justify left))
     )
-    (property "Footprint" "" (id 2) (at 66.04 30.48 0)
-      (effects (font (size 1.27 1.27)) hide)
-    )
+    (property "Footprint" "mio:MountingHole_3.2mm_M3" (id 2) (at 66.04 30.48 0)
+      (effects (font (size 1.27 1.27)) hide)
+    )
